Commit message: no-mistakes(review): Stamp commands with sim time, raise LiDAR min range

File: src/trashcan_description/urdf/properties.xacro (robot description, xacro)
@@ -6,5 +6,8 @@
 -->
 <robot xmlns:xacro="http://www.ros.org/wiki/xacro">
-  <!-- Drive wheels: 17 cm diameter, sized to climb a 5 cm (2 inch) step later. -->
+  <!--
+    Drive wheels: 17 cm diameter, a starting point for the 5 cm (2 inch) step.
+    Climbing it will also need its own caster and drive work.
+  -->
   <xacro:property name="wheel_radius" value="0.085"/>
   <xacro:property name="wheel_width" value="0.04"/>
@@ -25,5 +28,6 @@
   <xacro:property name="lidar_beam_z" value="0.19"/>
   <xacro:property name="lidar_mass" value="0.17"/>
-  <xacro:property name="lidar_min_range" value="0.12"/>
+  <!-- Beyond the bin posts, so the LiDAR does not see the robot itself. -->
+  <xacro:property name="lidar_min_range" value="0.15"/>
   <xacro:property name="lidar_max_range" value="12.0"/>
   <xacro:property name="lidar_samples" value="720"/>
